File: files/M3-RC.brd (EAGLE design)
At the start: 56.6 x 90 mm, 27 parts, among them U1 CR2032-BS-6-1

Commit message: Update files to RC
Parts:
- added U$1: UK000011, OSHWA:CERT-SMALL-SILK
Routing:
- net N$17: track 169.4 -> 176.2 mm
- net N$1: track 102.0 -> 105.9 mm
- net N$9: track 10.2 -> 12.1 mm
- net N$24: track 102.5 -> 104.0 mm
- net N$16: track 99.3 -> 98.2 mm
- net N$11: track 9.06 -> 9.76 mm
Other:
- board text added: "Leeds Raspberry Jam OTIS - Release Candidate"
- board text removed: "Final - Revision 3"
- board text removed: "LRJ Owl Badge"
